Commit message: Added paddle STL file and inserted it into UR10 URDF

File: urdf/ur10_robot.urdf (robot description, URDF)
Before this commit: robot ur10, 11 links, 10 joints
Links:
- added link paddle, mass 0.037; collision mesh filename=package://PingPongBot/urdf/paddle-Body.stl scale=0.001 0.001 0.001; visual mesh filename=package://PingPongBot/urdf/paddle-Body.stl scale=0.001 0.001 0.001
Joints:
- added joint paddle_fixed_joint: type fixed, parent tool0, child paddle, origin xyz=0 0 0.1 rpy=0 0 0

Commit message: Added Paddle to URDF and configured position/size

File: urdf/ur10_robot.urdf (robot description, URDF)
Before this commit: robot ur10, 12 links, 11 joints
Links:
- link paddle: geometry collision mesh filename=package://pingpongbot/urdf/paddle-Body.stl scale=0.002 0.002 0.002; visual mesh filename=package://pingpongbot/urdf/paddle-Body.stl scale=0.002 0.002 0.002
Joints:
- joint paddle_fixed_joint: origin xyz=0 0 0.1 rpy=0 0 0 -> xyz=0 0 0.15 rpy=0 0 0

Commit message: testing swing back sequence

File: urdf/ur10_robot.urdf (robot description, URDF)
Before this commit: robot ur10, 12 links, 11 joints
Links:
- added link tip
Joints:
- added joint tip_joint: type fixed, parent paddle, child tip, origin xyz=0 0 0 rpy=0 0 0

Commit message: fixed mesh loading

File: urdf/ur10_robot.urdf (robot description, URDF)
Before this commit: robot ur10, 13 links, 12 joints
Links:
- link base_link: geometry collision mesh filename=package://pingpongbot/meshes/ur10/collision/base.stl; visual mesh filename=package://pingpongbot/meshes/ur10/visual/base.dae
- link forearm_link: geometry collision mesh filename=package://pingpongbot/meshes/ur10/collision/forearm.stl; visual mesh filename=package://pingpongbot/meshes/ur10/visual/forearm.dae
- link shoulder_link: geometry collision mesh filename=package://pingpongbot/meshes/ur10/collision/shoulder.stl; visual mesh filename=package://pingpongbot/meshes/ur10/visual/shoulder.dae
- link upper_arm_link: geometry collision mesh filename=package://pingpongbot/meshes/ur10/collision/upperarm.stl; visual mesh filename=package://pingpongbot/meshes/ur10/visual/upperarm.dae
- link wrist_1_link: geometry collision mesh filename=package://pingpongbot/meshes/ur10/collision/wrist1.stl; visual mesh filename=package://pingpongbot/meshes/ur10/visual/wrist1.dae
- link wrist_2_link: geometry collision mesh filename=package://pingpongbot/meshes/ur10/collision/wrist2.stl; visual mesh filename=package://pingpongbot/meshes/ur10/visual/wrist2.dae
- link wrist_3_link: geometry collision mesh filename=package://pingpongbot/meshes/ur10/collision/wrist3.stl; visual mesh filename=package://pingpongbot/meshes/ur10/visual/wrist3.dae

Commit message: code refactoring

File: urdf/ur10_robot.urdf (robot description, URDF)
Before this commit: robot ur10, 13 links, 12 joints
Links:
- link base_link: geometry collision mesh filename=package://flyswatter/meshes/ur10/collision/base.stl; visual mesh filename=package://flyswatter/meshes/ur10/visual/base.dae
- link forearm_link: geometry collision mesh filename=package://flyswatter/meshes/ur10/collision/forearm.stl; visual mesh filename=package://flyswatter/meshes/ur10/visual/forearm.dae
- link paddle: geometry collision mesh filename=package://flyswatter/urdf/paddle-Body.stl scale=0.002 0.002 0.002; visual mesh filename=package://flyswatter/urdf/paddle-Body.stl scale=0.002 0.002 0.002
- link shoulder_link: geometry collision mesh filename=package://flyswatter/meshes/ur10/collision/shoulder.stl; visual mesh filename=package://flyswatter/meshes/ur10/visual/shoulder.dae
- link upper_arm_link: geometry collision mesh filename=package://flyswatter/meshes/ur10/collision/upperarm.stl; visual mesh filename=package://flyswatter/meshes/ur10/visual/upperarm.dae
- link wrist_1_link: geometry collision mesh filename=package://flyswatter/meshes/ur10/collision/wrist1.stl; visual mesh filename=package://flyswatter/meshes/ur10/visual/wrist1.dae
- link wrist_2_link: geometry collision mesh filename=package://flyswatter/meshes/ur10/collision/wrist2.stl; visual mesh filename=package://flyswatter/meshes/ur10/visual/wrist2.dae
- link wrist_3_link: geometry collision mesh filename=package://flyswatter/meshes/ur10/collision/wrist3.stl; visual mesh filename=package://flyswatter/meshes/ur10/visual/wrist3.dae
